Commit message: URDF name clank->alex

File: alex_description/urdf/20240109_Alex.noHands.urdf (robot description, URDF)
Before this commit: robot Alex, 21 links, 20 joints
Links:
- link Head: geometry visual mesh filename=package://alex_description/meshes/Head.obj
- link LeftElbowPitchLink: geometry visual mesh filename=package://alex_description/meshes/cycloidal_arm/LeftElbowPi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
- link LeftGripperYawLink: geometry visual mesh filename=package://alex_description/meshes/cycloidal_arm/LeftGripper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
- link LeftShoulderPitchLink: geometry visual mesh filename=package://alex_description/meshes/cycloidal_arm/LeftShoulde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
- link LeftShoulderRollLink: geometry visual mesh filename=package://alex_description/meshes/cycloidal_arm/LeftShoulde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
- link LeftShoulderYawLink: geometry visual mesh filename=package://alex_description/meshes/cycloidal_arm/LeftShoulde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
- link LeftWristRollLink: geometry visual mesh filename=package://alex_description/meshes/cycloidal_arm/LeftWristRo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
- link LeftWristYawLink: geometry visual mesh filename=package://alex_description/meshes/cycloidal_arm/LeftWristYa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
- link RightElbowPitchLink: geometry visual mesh filename=package://alex_description/meshes/cycloidal_arm/RightElbowP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
- link RightGripperYawLink: geometry visual mesh filename=package://alex_description/meshes/cycloidal_arm/RightGrippe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
- link RightShoulderPitchLink: geometry visual mesh filename=package://alex_description/meshes/cycloidal_arm/RightShould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
- link RightShoulderRollLink: geometry visual mesh filename=package://alex_description/meshes/cycloidal_arm/RightShould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
- link RightShoulderYawLink: geometry visual mesh filename=package://alex_description/meshes/cycloidal_arm/RightShould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
- link RightWristRollLink: geometry visual mesh filename=package://alex_description/meshes/cycloidal_arm/RightWristR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
- link RightWristYawLink: geometry visual mesh filename=package://alex_description/meshes/cycloidal_arm/RightWristY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
- link Torso: geometry visual mesh filename=package://alex_description/meshes/Torso.obj

Commit message: Fixed Shoulder Roll Zero Offset and Negative Inertia

File: alex_description/urdf/20240109_Alex.noHands.urdf (robot description, URDF)
Before this commit: robot Alex, 21 links, 20 joints
Joints:
- joint LeftShoulderPitch: origin xyz=-0.011 0.113 0.227 rpy=0.698132 0.0 0.0 -> xyz=-0.025 0.1 0.21449 rpy=0.698132 0.0 0.0
- joint LeftShoulderRoll: limit lower=-0.261799 upper=2.87979 effort=150.0 velocity=9.0 -> lower=-0.349066 upper=2.79253 effort=150.0 velocity=9.0; origin xyz=0.0 0.15676000 -0.01300000 rpy=-0.785398163 0.0 0.0 -> xyz=0.0 0.15676000 -0.01300000 rpy=-0.698132 0.0 0.0
- joint NeckPitch: limit lower=-1.0472 upper=1.0472 effort=20 velocity=20.0 -> lower=-1.0472 upper=1.0472 effort=20 velocity=20
- joint NeckYaw: limit lower=-1.5708 upper=1.5708 effort=80.0 velocity=20.0 -> lower=-1.5708 upper=1.5708 effort=20 velocity=20
- joint RightShoulderPitch: origin xyz=-0.011 -0.113 0.227 rpy=-0.698132 0.0 0.0 -> xyz=-0.025 -0.1 0.21449 rpy=-0.698132 0.0 0.0
- joint RightShoulderRoll: limit lower=-2.87979 upper=0.261799 effort=1000 velocity=100 -> lower=-2.79253 upper=0.349066 effort=1000 velocity=100; origin xyz=0.0 -0.15676000 -0.01300000 rpy=0.785398163 0.0 0.0 -> xyz=0.0 -0.15676000 -0.01300000 rpy=0.698132 0.0 0.0
- joint SpinePitch: limit lower=-0.785398 upper=0.785398 effort=200.0 velocity=6.0 -> lower=-0.523599 upper=1.0472 effort=250.0 velocity=6.0
- joint SpineYaw: limit lower=-1.0472 upper=1.0472 effort=80 velocity=20.0 -> lower=-1.0472 upper=1.0472 effort=150 velocity=9.0
