Commit message: Merged in feature/sakeHands (pull request #1)
Added a thin mesh of the Sake Hands and added an Alex Sake URDF model

* Added a thin mesh of the Sake Hands and added an Alex Sake URDF model

Added the sake meshes to sake_description
Depolygonized the palm link
finger meshes could still be optimized more
added 20240109_Alex_SakeHands.urdf
TODO: add xacros / composite builds off URDFs

* added nub hands and a nub urdf
* changed ability_hand_description folder name hyphens to lowercase

Approved-by: Achintya Mohan

File: alex_description/urdf/20240109_Alex_PsyonicHands.urdf (robot description, URDF)
Before this commit: robot Alex, 55 links, 54 joints
Links:
- link LeftPsyonicAbilityBaseLink: geometry visual mesh filename=package://ability_hand_description/models/wristmesh.obj
- link Left_index_L1: geometry visual mesh filename=package://ability_hand_description/models/idx-f1.obj
- link Left_index_L2: geometry visual mesh filename=package://ability_hand_description/models/idx-f2.obj
- link Left_middle_L1: geometry visual mesh filename=package://ability_hand_description/models/idx-f1.obj
- link Left_middle_L2: geometry visual mesh filename=package://ability_hand_description/models/idx-f2.obj
- link Left_pinky_L1: geometry visual mesh filename=package://ability_hand_description/models/idx-f1.obj
- link Left_pinky_L2: geometry visual mesh filename=package://ability_hand_description/models/idx-f2.obj
- link Left_ring_L1: geometry visual mesh filename=package://ability_hand_description/models/idx-f1.obj
- link Left_ring_L2: geometry visual mesh filename=package://ability_hand_description/models/idx-f2.obj
- link Left_thumb_L1: geometry visual mesh filename=package://ability_hand_description/models/thumb-f1.obj
- link Left_thumb_L2: geometry visual mesh filename=package://ability_hand_description/models/thumb-f2-left.obj
- link Left_thumb_base: geometry visual mesh filename=package://ability_hand_description/models/fb_palm_ref.obj
- link RightPsyonicAbilityBaseLink: geometry visual mesh filename=package://ability_hand_description/models/wristmesh.obj
- link Right_index_L1: geometry visual mesh filename=package://ability_hand_description/models/idx-f1.obj
- link Right_index_L2: geometry visual mesh filename=package://ability_hand_description/models/idx-f2.obj
- link Right_middle_L1: geometry visual mesh filename=package://ability_hand_description/models/idx-f1.obj
- link Right_middle_L2: geometry visual mesh filename=package://ability_hand_description/models/idx-f2.obj
- link Right_pinky_L1: geometry visual mesh filename=package://ability_hand_description/models/idx-f1.obj
- link Right_pinky_L2: geometry visual mesh filename=package://ability_hand_description/models/idx-f2.obj
- link Right_ring_L1: geometry visual mesh filename=package://ability_hand_description/models/idx-f1.obj
- link Right_ring_L2: geometry visual mesh filename=package://ability_hand_description/models/idx-f2.obj
- link Right_thumb_L1: geometry visual mesh filename=package://ability_hand_description/models/thumb-f1-mir.obj
- link Right_thumb_L2: geometry visual mesh filename=package://ability_hand_description/models/thumb-f2-right.obj
- link Right_thumb_base: geometry visual mesh filename=package://ability_hand_description/models/fb_palm_ref_mir.o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
