Commit message: Best guess on torso offset for now.

File: alex_description/urdf/20240516_Alex_TwoArms_SakeHands.urdf (robot description, URDF)
Before this commit: robot Alex, 25 links, 24 joints
Links:
- link Pelvis: geometry visual mesh filename=package://alex_description/meshes/Torso_Base_and_Head.obj

Commit message: Adjusted the offsets with Sam

File: alex_description/urdf/20240516_Alex_TwoArms_SakeHands.urdf (robot description, URDF)
Before this commit: robot Alex, 25 links, 24 joints
Joints:
- joint LeftShoulderPitch: origin xyz=-0.025 0.1 0.550 rpy=0.698132 0.0 0.0 -> xyz=0.0 0.1 0.570 rpy=0.698132 0.0 0.0
- joint RightShoulderPitch: origin xyz=-0.025 -0.1 0.550 rpy=-0.698132 0.0 0.0 -> xyz=0.0 -0.1 0.570 rpy=-0.698132 0.0 0.0

Commit message: Adjusted x offset

File: alex_description/urdf/20240516_Alex_TwoArms_SakeHands.urdf (robot description, URDF)
Before this commit: robot Alex, 25 links, 24 joints
Joints:
- joint LeftShoulderPitch: origin xyz=0.0 0.1 0.570 rpy=0.698132 0.0 0.0 -> xyz=-0.0114 0.1 0.570 rpy=0.698132 0.0 0.0
- joint RightShoulderPitch: origin xyz=0.0 -0.1 0.570 rpy=-0.698132 0.0 0.0 -> xyz=-0.0114 -0.1 0.570 rpy=-0.698132 0.0 0.0

Commit message: Removed the bicep extension from the urdf.

File: alex_description/urdf/20240516_Alex_TwoArms_SakeHands.urdf (robot description, URDF)
Before this commit: robot Alex, 25 links, 24 joints
Links:
- link LeftShoulderRollLink: mass 1.17068 -> 0.971
- link RightShoulderRollLink: mass 1.17068 -> 0.971
Joints:
- joint LeftElbowPitch: origin xyz=0.015 0.0 -0.4 rpy=0.0 0.0 0.0 -> xyz=0.015 0.0 -0.3127 rpy=0.0 0.0 0.0
- joint RightElbowPitch: origin xyz=0.015 0.0 -0.4 rpy=0.0 0.0 0.0 -> xyz=0.015 0.0 -0.3127 rpy=0.0 0.0 0.0
