Commit message: Adjusted Psyoinic retargeting parameters for VR and fixed joints in the urdf.

File: alex_description/urdf/20240619_Alex_TestStand_Fixed_Head_PsyonicHands.urdf (robot description, URDF)
Before this commit: robot Alex, 49 links, 48 joints
Joints:
- joint Left_index_q1: type revolute -> fixed
- joint Left_index_q2: type revolute -> fixed
- joint Left_middle_q1: type revolute -> fixed
- joint Left_middle_q2: type revolute -> fixed
- joint Left_pinky_q1: type revolute -> fixed
- joint Left_pinky_q2: type revolute -> fixed
- joint Left_ring_q1: type revolute -> fixed
- joint Left_ring_q2: type revolute -> fixed
- joint Left_thumb_q1: type revolute -> fixed
- joint Left_thumb_q2: type revolute -> fixed
- joint Right_index_q1: type revolute -> fixed
- joint Right_index_q2: type revolute -> fixed
- joint Right_middle_q1: type revolute -> fixed
- joint Right_middle_q2: type revolute -> fixed
- joint Right_pinky_q1: type revolute -> fixed
- joint Right_pinky_q2: type revolute -> fixed
- joint Right_ring_q1: type revolute -> fixed
- joint Right_ring_q2: type revolute -> fixed
- joint Right_thumb_q1: type revolute -> fixed
- joint Right_thumb_q2: type revolute -> fixed
