Commit message: Merged feature/alex-ui into develop

File: alex_description/urdf/20240109_Alex_SakeHands.urdf (robot description, URDF)
Before this commit: robot Alex, 31 links, 30 joints
Links:
- added link LeftShoulderPitchIMULink, mass 0
- added link LeftShoulderYawIMULink, mass 0
- added link LeftWristYawIMULink, mass 0
- link LeftGripperYawLink: mass 0.2480 -> 0.3
- link LeftWristRollLink: mass 0.6953487750589724 -> 0.874
- link LeftWristYawLink: mass 1.5075249788801466 -> 1.438
- link RightGripperYawLink: mass 0.2480 -> 0.3
Joints:
- added joint LeftShoulderPitchIMUJoint: type fixed, parent LeftShoulderPitchLink, child LeftShoulderPitchIMULink, origin xyz=0.0174 0.06944 -0.03025 rpy=-1.570796 1.570796 0, axis 0 0 1
- added joint LeftShoulderYawIMUJoint: type fixed, parent LeftShoulderYawLink, child LeftShoulderYawIMULink, origin xyz=-0.00763459 -0.0123324 -0.318 rpy=-1.570796 3.1415926 -0.314159, axis 0 0 1
- added joint LeftWristYawIMUJoint: type fixed, parent LeftWristYawLink, child LeftWristYawIMULink, origin xyz=-0.033554 0.010450 -0.148527 rpy=1.571  0.0 1.571, axis 0 0 1

Commit message: Added reachability trajectories. Fixed the fingers on the sake hands.

File: alex_description/urdf/20240109_Alex_SakeHands.urdf (robot description, URDF)
Before this commit: robot Alex, 34 links, 33 joints
Joints:
- joint LeftSakeBaseFingerJoint1: type revolute -> fixed
- joint LeftSakeBaseFingerJoint2: type revolute -> fixed
- joint LeftSakeKnuckle1: type revolute -> fixed
- joint LeftSakeKnuckle2: type revolute -> fixed
- joint RightSakeBaseFingerJoint1: type revolute -> fixed
- joint RightSakeBaseFingerJoint2: type revolute -> fixed
- joint RightSakeKnuckle1: type revolute -> fixed
- joint RightSakeKnuckle2: type revolute -> fixed

File: alex_description/urdf/20240516_Alex_TestStand_Fixed_Head.urdf (robot description, URDF)
Before this commit: robot Alex, 25 links, 24 joints
Joints:
- joint LeftSakeBaseFingerJoint1: type revolute -> fixed
- joint LeftSakeBaseFingerJoint2: type revolute -> fixed
- joint LeftSakeKnuckle1: type revolute -> fixed
- joint LeftSakeKnuckle2: type revolute -> fixed
- joint RightSakeBaseFingerJoint1: type revolute -> fixed
- joint RightSakeBaseFingerJoint2: type revolute -> fixed
- joint RightSakeKnuckle1: type revolute -> fixed
- joint RightSakeKnuckle2: type revolute -> fixed

Commit message: added URDF's with updated IMU locations

File: alex_description/urdf/20240109_Alex_SakeHands.urdf (robot description, URDF)
Before this commit: robot Alex, 34 links, 33 joints
Links:
- removed link PelvisStimIMUMount
Joints:
- removed joint PelvisStimIMUFixedJoint

File: alex_description/urdf/20240619_Alex_TestStand_FixedHead_PsyonicHands.urdf (robot description, URDF)
Before this commit: robot Alex, 49 links, 48 joints
Links:
- added link LeftShoulderPitchIMULink, mass 0
- added link LeftShoulderYawIMULink, mass 0
- added link LeftWristYawIMULink, mass 0
- added link RightShoulderPitchIMULink, mass 0
- added link RightShoulderYawIMULink, mass 0
- added link RightWristYawIMULink, mass 0
- added link TorsoLeftIMULink, mass 0
- added link TorsoRightIMULink, mass 0
Joints:
- added joint LeftShoulderPitchIMUJoint: type fixed, parent LeftShoulderPitchLink, child LeftShoulderPitchIMULink, origin xyz=0.01432621 0.0755071 -0.00245783 rpy=-3.141592 0 -1.57079632679, axis 0 0 1
- added joint LeftShoulderYawIMUJoint: type fixed, parent LeftShoulderYawLink, child LeftShoulderYawIMULink, origin xyz=-0.00633723 -0.00669505 -0.19881468 rpy=1.570796 3.1415926 -0.314159, axis 0 0 1
- added joint LeftWristYawIMUJoint: type fixed, parent LeftWristYawLink, child LeftWristYawIMULink, origin xyz=-0.033986 0.011658 -0.148527 rpy=1.571  0.0 1.571, axis 0 0 1
- added joint RightShoulderPitchIMUJoint: type fixed, parent RightShoulderPitchLink, child RightShoulderPitchIMULink, origin xyz=0.01432621 -0.10001299 -0.00245783 rpy=3.141592 0 -1.57079632679, axis 0 0 1
- added joint RightShoulderYawIMUJoint: type fixed, parent RightShoulderYawLink, child RightShoulderYawIMULink, origin xyz=0.00119168 0.00914134 -0.19881468 rpy=-1.570796 0.0 0.314159, axis 0 0 1
- added joint RightWristYawIMUJoint: type fixed, parent RightWristYawLink, child RightWristYawIMULink, origin xyz=-0.033986 0.011658 -0.148527 rpy=1.571  0.0 1.571, axis 0 0 1
- added joint TorsoLeftIMUJoint: type fixed, parent Pelvis, child TorsoLeftIMULink, origin xyz=-0.102655 0.034047 0.488646 rpy=1.570796 0 -1.570796, axis 0 0 1
- added joint TorsoRightIMUJoint: type fixed, parent Pelvis, child TorsoRightIMULink, origin xyz=-0.105655 -0.059053 0.488646 rpy=1.570796 0 -1.570796, axis 0 0 1
