Commit message: Updated URDF with thorough CAD verification
Found a bug with the Shoulder yaw COM position

File: alex_description/urdf/20240619_Alex_TestStand_FixedHead_NoHands.urdf (robot description, URDF)
Before this commit: robot Alex, 23 links, 22 joints
Links:
- link RightElbowPitchLink: mass 0.4895385722366345 -> 0.45
- link RightGripperYawLink: mass 0.2480 -> 0.251
- link RightShoulderPitchLink: mass 2.917 -> 2.99
- link RightShoulderRollLink: mass 0.971 -> 0.972
- link RightShoulderYawLink: mass 2.53059 -> 2.91
- link RightWristRollLink: mass 0.874 -> 0.909
- link RightWristYawLink: mass 1.438 -> 1.547
