Commit message: Updated pysonic URDF
Fixed the J3 COM bug and verfied with CAD

File: alex_description/urdf/20240619_Alex_TestStand_FixedHead_PsyonicHands.urdf (robot description, URDF)
Before this commit: robot Alex, 57 links, 56 joints
Links:
- link RightElbowPitchLink: mass 0.4895385722366345 -> 0.45
- link RightGripperYawLink: mass 0.2480 -> 0.251
- link RightShoulderPitchLink: mass 2.917 -> 2.99
- link RightShoulderRollLink: mass 0.971 -> 0.972
- link RightShoulderYawLink: mass 2.53059 -> 2.91
- link RightWristRollLink: mass 0.874 -> 0.909
- link RightWristYawLink: mass 1.438 -> 1.547
Joints:
- joint RightWristYawIMUJoint: origin xyz=-0.033986 0.011658 -0.148527 rpy=1.571  0.0 1.571 -> xyz=-0.048986 0.011658 -0.149476 rpy=1.571  0.0 1.571
