Commit message: Adjusted barrett placeholder inertias.

File: alex_description/urdf/20240614_Alex_TestStand_FixedHead_BarrettDumbbell.urdf (robot description, URDF)
Before this commit: robot Alex, 24 links, 23 joints
Links:
- removed link bh280/finger0_0
- removed link bh280/finger0_1
- removed link bh280/finger0_2
- removed link bh280/hand_base
- added link RightBarrettPalmLink, mass 0.944
- added link RightHandDumbbellLink, mass 2.676
Joints:
- removed joint bh280/j00
- removed joint bh280/j01
- removed joint bh280/j02
- added joint RightHandDumbbellAttachmentFixedJoint: type fixed, parent RightBarrettPalmLink, child RightHandDumbbellLink, origin xyz=0 0 -0.027 rpy=0 0 0
- joint RightGrippertAttachmentFixedJoint: child bh280/hand_base -> RightBarrettPalmLink

Commit message: Changes needed for hardware testing: 1) switched to using the left hand in weight trajectories, 2) adjusted urdf, hand version, and kinematics collisions to use the left hand.

File: alex_description/urdf/20240614_Alex_TestStand_FixedHead_BarrettDumbbell.urdf (robot description, URDF)
Before this commit: robot Alex, 22 links, 21 joints
Links:
- removed link LeftSakeBaseFingerLink1
- removed link LeftSakeBaseFingerLink2
- removed link LeftSakeFingerTip1
- removed link LeftSakeFingerTip2
- removed link LeftSakePalmLink
- removed link RightHandDumbbellLink
- added link LeftBarrettPalmLink, mass 0.944
Joints:
- removed joint LeftSakeBaseFingerJoint1
- removed joint LeftSakeBaseFingerJoint2
- removed joint LeftSakeKnuckle1
- removed joint LeftSakeKnuckle2
- removed joint RightHandDumbbellAttachmentFixedJoint
- joint LeftGrippertAttachmentFixedJoint: child LeftSakePalmLink -> LeftBarrettPalmLink

Commit message: Adjusted barret orientation to match hardware. There were some cascading changes to scripted trajectories.

File: alex_description/urdf/20240614_Alex_TestStand_FixedHead_BarrettDumbbell.urdf (robot description, URDF)
Before this commit: robot Alex, 17 links, 16 joints
Links:
- added link LeftHandDumbbellLink, mass 3.956
Joints:
- added joint LeftHandDumbbellAttachmentFixedJoint: type fixed, parent LeftBarrettPalmLink, child LeftHandDumbbellLink, origin xyz=0 0 -0.027 rpy=0 0 0

Commit message: Changed default version to Barrett hands with dumbbells and uncommented them in the urdf. Changed damping gain in acceleration integration to be higher by default to improve tracking. (Christian)

File: alex_description/urdf/20240614_Alex_TestStand_FixedHead_BarrettDumbbell.urdf (robot description, URDF)
Before this commit: robot Alex, 18 links, 17 joints
Links:
- added link RightHandDumbbellLink, mass 3.956
Joints:
- added joint RightHandDumbbellAttachmentFixedJoint: type fixed, parent RightBarrettPalmLink, child RightHandDumbbellLink, origin xyz=0 0 -0.027 rpy=0 0 0

Commit message: Removed dumbbell inertia.

File: alex_description/urdf/20240614_Alex_TestStand_FixedHead_BarrettDumbbell.urdf (robot description, URDF)
Before this commit: robot Alex, 19 links, 18 joints
Links:
- removed link LeftHandDumbbellLink
- removed link RightHandDumbbellLink
Joints:
- removed joint LeftHandDumbbellAttachmentFixedJoint
- removed joint RightHandDumbbellAttachmentFixedJoint

Commit message: Fixed dumbbell inertia orientation to make sense with the barrett hand orientation.

File: alex_description/urdf/20240614_Alex_TestStand_FixedHead_BarrettDumbbell.urdf (robot description, URDF)
Before this commit: robot Alex, 17 links, 16 joints
Links:
- link LeftBarrettPalmLink: geometry visual mesh filename=package://barrett_description/meshes/bh280/hand_base.dae
- link RightBarrettPalmLink: geometry visual mesh filename=package://barrett_description/meshes/bh280/hand_base.dae

Commit message: Updated shoulder roll meshes and fixed the name of an enum.

File: alex_description/urdf/20240614_Alex_TestStand_FixedHead_BarrettDumbbell.urdf (robot description, URDF)
Before this commit: robot Alex, 17 links, 16 joints
Links:
- link LeftBarrettPalmLink: geometry 
- link RightBarrettPalmLink: geometry 

Commit message: Updated barett and psyonic hands urdfs

File: alex_description/urdf/20240614_Alex_TestStand_FixedHead_BarrettDumbbell.urdf (robot description, URDF)
Before this commit: robot Alex, 17 links, 16 joints
Links:
- removed link LeftBarrettPalmLink
- added link LeftShoulderPitchIMULink, mass 0
- added link LeftShoulderYawIMULink, mass 0
- added link LeftWristYawIMULink, mass 0
- added link RightHandDumbbellLink, mass 3.956
- added link RightShoulderPitchIMULink, mass 0
- added link RightShoulderYawIMULink, mass 0
- added link RightWristYawIMULink, mass 0
- link LeftWristRollLink: mass 0.6953487750589724 -> 0.874
- link LeftWristYawLink: mass 1.5075249788801466 -> 1.438
- link RightBarrettPalmLink: geometry visual mesh filename=package://barrett_description/meshes/bh280/hand_base.dae
- link RightWristRollLink: mass 0.6953487750589724 -> 0.874
- link RightWristYawLink: mass 1.5075249788801466 -> 1.438
Joints:
- removed joint LeftGrippertAttachmentFixedJoint
- added joint LeftShoulderPitchIMUJoint: type fixed, parent LeftShoulderPitchLink, child LeftShoulderPitchIMULink, origin xyz=0.01432621 0.0755071 -0.00245783 rpy=-3.141592 0 -1.57079632679, axis 0 0 1
- added joint LeftShoulderYawIMUJoint: type fixed, parent LeftShoulderYawLink, child LeftShoulderYawIMULink, origin xyz=-0.00633723 -0.00669505 -0.19881468 rpy=1.570796 3.1415926 -0.314159, axis 0 0 1
- added joint LeftWristYawIMUJoint: type fixed, parent LeftWristYawLink, child LeftWristYawIMULink, origin xyz=-0.048986 0.011658 -0.149476 rpy=1.571  0.0 1.571, axis 0 0 1
- added joint RightHandDumbbellAttachmentFixedJoint: type fixed, parent RightBarrettPalmLink, child RightHandDumbbellLink, origin xyz=0 0 -0.027 rpy=0 0 0
- added joint RightShoulderPitchIMUJoint: type fixed, parent RightShoulderPitchLink, child RightShoulderPitchIMULink, origin xyz=0.01432621 -0.10001299 -0.00245783 rpy=3.141592 0 -1.57079632679, axis 0 0 1
- added joint RightShoulderYawIMUJoint: type fixed, parent RightShoulderYawLink, child RightShoulderYawIMULink, origin xyz=0.00119168 0.00914134 -0.19881468 rpy=-1.570796 0.0 0.314159, axis 0 0 1
- added joint RightWristYawIMUJoint: type fixed, parent RightWristYawLink, child RightWristYawIMULink, origin xyz=-0.048986 0.011658 -0.149476 rpy=1.571  0.0 1.571, axis 0 0 1

File: alex_description/urdf/20240619_Alex_TestStand_FixedHead_PsyonicHands.urdf (robot description, URDF)
Before this commit: robot Alex, 57 links, 56 joints
Links:
- link LeftWristRollLink: mass 0.6953487750589724 -> 0.874
- link LeftWristYawLink: mass 1.5075249788801466 -> 1.438
- link RightWristRollLink: mass 0.6953487750589724 -> 0.874
- link RightWristYawLink: mass 1.5075249788801466 -> 1.438
Joints:
- joint LeftWristYawIMUJoint: origin xyz=-0.033986 0.011658 -0.148527 rpy=1.571  0.0 1.571 -> xyz=-0.048986 0.011658 -0.149476 rpy=1.571  0.0 1.571

Commit message: Updated left arm masses on URDF models

File: alex_description/urdf/20240614_Alex_TestStand_FixedHead_BarrettDumbbell.urdf (robot description, URDF)
Before this commit: robot Alex, 23 links, 22 joints
Links:
- link LeftGripperYawLink: mass 0.2480 -> 0.251
- link LeftShoulderPitchLink: mass 2.917 -> 3.025
- link LeftShoulderYawLink: mass 2.53059 -> 2.93
- link LeftWristRollLink: mass 0.874 -> 0.909
- link LeftWristYawLink: mass 1.438 -> 1.55

File: alex_description/urdf/20240619_Alex_TestStand_FixedHead_NoHands.urdf (robot description, URDF)
Before this commit: robot Alex, 23 links, 22 joints
Links:
- link LeftGripperYawLink: mass 0.2480 -> 0.251
- link LeftShoulderPitchLink: mass 2.917 -> 3.025
- link LeftShoulderYawLink: mass 2.53059 -> 2.93
- link LeftWristRollLink: mass 0.874 -> 0.909
- link LeftWristYawLink: mass 1.438 -> 1.55

File: alex_description/urdf/20240619_Alex_TestStand_FixedHead_PsyonicHands.urdf (robot description, URDF)
Before this commit: robot Alex, 57 links, 56 joints
Links:
- link LeftGripperYawLink: mass 0.2480 -> 0.251
- link LeftShoulderPitchLink: mass 2.917 -> 3.025
- link LeftShoulderYawLink: mass 2.53059 -> 2.93
- link LeftWristRollLink: mass 0.874 -> 0.909
- link LeftWristYawLink: mass 1.438 -> 1.55

Commit message: Commented out the visual since RDX can't handle the file type.

File: alex_description/urdf/20240614_Alex_TestStand_FixedHead_BarrettDumbbell.urdf (robot description, URDF)
Before this commit: robot Alex, 23 links, 22 joints
Links:
- link RightBarrettPalmLink: geometry 
