Commit message: Updated nub Hands URDF

File: alex_description/urdf/20240109_Alex_nubHands.urdf (robot description, URDF)
Before this commit: robot Alex, 23 links, 22 joints
Joints:
- joint leftGrippertAttachmentFixedJoint: child rightNub -> leftNub
- joint rightGrippertAttachmentFixedJoint: child leftNub -> rightNub
