Commit message: Fixed bug in Psyonic hand URDF

File: alex_description/urdf/20240808_Alex_Spineless_PsyonicHands.urdf (robot description, URDF)
Before this commit: robot Alex, 27 links, 26 joints
Links:
- link LeftPsyonicHand: geometry visual mesh filename=package://ability_hand_description/models/PsyonicLeft.obj
- link RightPsyonicHand: geometry visual mesh filename=package://ability_hand_description/models/PsyonicRight.obj
Joints:
- joint LeftGrippertAttachmentFixedJoint: type revolute -> fixed
- joint RightGrippertAttachmentFixedJoint: type revolute -> fixed
