Commit message: Updated UDFs

File: alex_description/urdf/20240808_Alex_Spineless_Nubs.urdf (robot description, URDF)
Before this commit: robot Alex, 25 links, 24 joints
Links:
- added link leftNub, mass 0.1; visual mesh filename=package://alex_description/meshes/cycloidal_arm/nub.obj
- added link rightNub, mass 0.1; visual mesh filename=package://alex_description/meshes/cycloidal_arm/nub.obj
- link NeckYawLink: mass 1.0 -> 0.708
- link Pelvis: geometry visual mesh filename=package://alex_description/meshes/TorsoFixedBaseWithoutSpin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
Joints:
- added joint LeftGrippertAttachmentFixedJoint: type fixed, parent LeftGripperYawLink, child leftNub, origin xyz=0 0 -0.0210000 rpy=0 0 0
- added joint RightGrippertAttachmentFixedJoint: type fixed, parent RightGripperYawLink, child rightNub, origin xyz=0 0 -0.0210000 rpy=0 0 0
- joint NeckPitch: origin xyz=0.025 0.0 0.173 rpy=0 0 0 -> xyz=0.025 -0.027544 0.245212 rpy=0 0 0
- joint NeckYaw: origin xyz=0.0 0.0 0.692 rpy=0 0 0 -> xyz=0.000094 -0.000003 0.625793 rpy=0 0 0

File: alex_description/urdf/20240808_Alex_WithSpine_Nubs.urdf (robot description, URDF)
Before this commit: robot Alex, 25 links, 24 joints
Links:
- added link SpineRollLink, mass 0.44
- added link SpineYawLink, mass 0.91
- added link Torso, mass 13.5; visual mesh filename=package://alex_description/meshes/Torso.obj
- added link leftNub, mass 0.1; visual mesh filename=package://alex_description/meshes/cycloidal_arm/nub.obj
- added link rightNub, mass 0.1; visual mesh filename=package://alex_description/meshes/cycloidal_arm/nub.obj
- link NeckYawLink: mass 1.0 -> 0.708
- link Pelvis: geometry visual mesh filename=package://alex_description/meshes/Torso.obj
Joints:
- added joint LeftGrippertAttachmentFixedJoint: type fixed, parent LeftGripperYawLink, child leftNub, origin xyz=0 0 -0.0210000 rpy=0 0 0
- added joint RightGrippertAttachmentFixedJoint: type fixed, parent RightGripperYawLink, child rightNub, origin xyz=0 0 -0.0210000 rpy=0 0 0
- added joint SpinePitch: type revolute, parent SpineRollLink, child Torso, origin xyz=0.12 0.0 0.0 rpy=0 0 0, axis 0 1 0, limit lower=-0.523599 upper=1.0472 effort=250.0 velocity=6.0
- added joint SpineRoll: type revolute, parent SpineYawLink, child SpineRollLink, origin xyz=-0.08 0 0.12 rpy=0 0 0, axis 1 0 0, limit lower=-0.436332 upper=0.436332 effort=150.0 velocity=6.0
- added joint SpineYaw: type revolute, parent Pelvis, child SpineYawLink, origin xyz=-0.129 0 0.35 rpy=0 0 0, axis 0 0 1, limit lower=-1.0472 upper=1.0472 effort=150 velocity=9.0
- joint LeftShoulderPitch: parent Pelvis -> Torso
- joint NeckPitch: origin xyz=0.025 0.0 0.173 rpy=0 0 0 -> xyz=0.025 -0.027544 0.245212 rpy=0 0 0
- joint NeckYaw: origin xyz=0.0 0.0 0.692 rpy=0 0 0 -> xyz=-0.089094 0.00003 0.324207 rpy=0 0 0; parent Pelvis -> Torso
- joint RightShoulderPitch: parent Pelvis -> Torso
