Commit message: Updated URDFs

File: alex_description/urdf/20240808_Alex_WithSpine_Nubs.urdf (robot description, URDF)
Before this commit: robot Alex, 30 links, 29 joints
Links:
- link Pelvis: geometry 
Joints:
- joint LeftShoulderPitch: origin xyz=-0.0114 0.1 0.570 rpy=0.698132 0.0 0.0 -> xyz=-0.025 0.1 0.214 rpy=0.698132 0.0 0.0
- joint NeckYaw: origin xyz=-0.089094 0.00003 0.324207 rpy=0 0 0 -> xyz=0.0 -0.00003 0.275793 rpy=0 0 0
- joint RightShoulderPitch: origin xyz=-0.0114 -0.1 0.570 rpy=-0.698132 0.0 0.0 -> xyz=-0.025 -0.1 0.214 rpy=-0.698132 0.0 0.0
