Commit message: Made some sake joints revolute

File: alex_description/urdf/20240808_Alex_FixedSpine_SakeHands.urdf (robot description, URDF)
Before this commit: robot Alex, 35 links, 34 joints
Joints:
- joint LeftSakeBaseFingerJoint1: type fixed -> revolute
- joint LeftSakeBaseFingerJoint2: type fixed -> revolute
- joint RightSakeBaseFingerJoint1: type fixed -> revolute
- joint RightSakeBaseFingerJoint2: type fixed -> revolute

Commit message: Fixed bugs in code

File: alex_description/urdf/20240808_Alex_FixedSpine_SakeHands.urdf (robot description, URDF)
Before this commit: robot Alex, 35 links, 34 joints
Joints:
- removed joint LeftSakeBaseFingerJoint1
- removed joint LeftSakeBaseFingerJoint2
- removed joint RightSakeBaseFingerJoint1
- removed joint RightSakeBaseFingerJoint2
- added joint Left_GRIPPER_X1: type revolute, parent LeftSakePalmLink, child LeftSakeBaseFingerLink1, origin xyz=0.0 0.0299 -0.0754 rpy=-0.25 0.0 0.0, axis 1.0 0.0 0.0, limit lower=-0.06 upper=1.9 effort=1.0 velocity=3.67
- added joint Left_GRIPPER_X2: type revolute, parent LeftSakePalmLink, child LeftSakeBaseFingerLink2, origin xyz=0.0 -0.0299 -0.0754 rpy=0.25 0.0 0.0, axis -1.0 0.0 0.0, limit lower=-0.06 upper=1.9 effort=1.0 velocity=3.67
- added joint Right_GRIPPER_X1: type revolute, parent RightSakePalmLink, child RightSakeBaseFingerLink1, origin xyz=0.0 0.0299 -0.0754 rpy=-0.25 0.0 0.0, axis 1.0 0.0 0.0, limit lower=-0.06 upper=1.9 effort=1.0 velocity=3.67
- added joint Right_GRIPPER_X2: type revolute, parent RightSakePalmLink, child RightSakeBaseFingerLink2, origin xyz=0.0 -0.0299 -0.0754 rpy=0.25 0.0 0.0, axis -1.0 0.0 0.0, limit lower=-0.06 upper=1.9 effort=1.0 velocity=3.67
