Commit message: Adjusted neck yaw and shoulder pitch offsets after test stand shortening.

File: alex_description/urdf/20240808_Alex_FixedSpine_BarrettHands.urdf (robot description, URDF)
Before this commit: robot Alex, 38 links, 36 joints
Joints:
- joint LeftShoulderPitch: origin xyz=-0.0114 0.1 0.570 rpy=0.698132 0.0 0.0 -> xyz=-0.0114 0.1 0.407 rpy=0.698132 0.0 0.0
- joint NeckYaw: origin xyz=0.000094 -0.000003 0.625793 rpy=0 0 0 -> xyz=0.000094 -0.000003 0.462793 rpy=0 0 0
- joint RightShoulderPitch: origin xyz=-0.0114 -0.1 0.570 rpy=-0.698132 0.0 0.0 -> xyz=-0.0114 -0.1 0.407 rpy=-0.698132 0.0 0.0

File: alex_description/urdf/20240808_Alex_FixedSpine_NoHands.urdf (robot description, URDF)
Before this commit: robot Alex, 27 links, 26 joints
Joints:
- joint LeftShoulderPitch: origin xyz=-0.0114 0.1 0.570 rpy=0.698132 0.0 0.0 -> xyz=-0.0114 0.1 0.407 rpy=0.698132 0.0 0.0
- joint NeckYaw: origin xyz=0.000094 -0.000003 0.625793 rpy=0 0 0 -> xyz=0.000094 -0.000003 0.462793 rpy=0 0 0
- joint RightShoulderPitch: origin xyz=-0.0114 -0.1 0.570 rpy=-0.698132 0.0 0.0 -> xyz=-0.0114 -0.1 0.407 rpy=-0.698132 0.0 0.0

File: alex_description/urdf/20240808_Alex_FixedSpine_Nubs.urdf (robot description, URDF)
Before this commit: robot Alex, 27 links, 26 joints
Joints:
- joint LeftShoulderPitch: origin xyz=-0.0114 0.1 0.570 rpy=0.698132 0.0 0.0 -> xyz=-0.0114 0.1 0.407 rpy=0.698132 0.0 0.0
- joint NeckYaw: origin xyz=0.000094 -0.000003 0.625793 rpy=0 0 0 -> xyz=0.000094 -0.000003 0.462793 rpy=0 0 0
- joint RightShoulderPitch: origin xyz=-0.0114 -0.1 0.570 rpy=-0.698132 0.0 0.0 -> xyz=-0.0114 -0.1 0.407 rpy=-0.698132 0.0 0.0

File: alex_description/urdf/20240808_Alex_FixedSpine_PsyonicHands.urdf (robot description, URDF)
Before this commit: robot Alex, 27 links, 26 joints
Joints:
- joint LeftShoulderPitch: origin xyz=-0.0114 0.1 0.570 rpy=0.698132 0.0 0.0 -> xyz=-0.0114 0.1 0.407 rpy=0.698132 0.0 0.0
- joint NeckYaw: origin xyz=0.000094 -0.000003 0.625793 rpy=0 0 0 -> xyz=0.000094 -0.000003 0.462793 rpy=0 0 0
- joint RightShoulderPitch: origin xyz=-0.0114 -0.1 0.570 rpy=-0.698132 0.0 0.0 -> xyz=-0.0114 -0.1 0.407 rpy=-0.698132 0.0 0.0

File: alex_description/urdf/20240808_Alex_FixedSpine_RightBarettWithWeights_LeftSake.urdf (robot description, URDF)
Before this commit: robot Alex, 43 links, 40 joints
Joints:
- joint LeftShoulderPitch: origin xyz=-0.0114 0.1 0.570 rpy=0.698132 0.0 0.0 -> xyz=-0.0114 0.1 0.407 rpy=0.698132 0.0 0.0
- joint NeckYaw: origin xyz=0.000094 -0.000003 0.625793 rpy=0 0 0 -> xyz=0.000094 -0.000003 0.462793 rpy=0 0 0
- joint RightShoulderPitch: origin xyz=-0.0114 -0.1 0.570 rpy=-0.698132 0.0 0.0 -> xyz=-0.0114 -0.1 0.407 rpy=-0.698132 0.0 0.0

File: alex_description/urdf/20240808_Alex_FixedSpine_SakeHands.urdf (robot description, URDF)
Before this commit: robot Alex, 35 links, 34 joints
Joints:
- joint LeftShoulderPitch: origin xyz=-0.0114 0.1 0.570 rpy=0.698132 0.0 0.0 -> xyz=-0.0114 0.1 0.407 rpy=0.698132 0.0 0.0
- joint NeckYaw: origin xyz=0.000094 -0.000003 0.625793 rpy=0 0 0 -> xyz=0.000094 -0.000003 0.462793 rpy=0 0 0
- joint RightShoulderPitch: origin xyz=-0.0114 -0.1 0.570 rpy=-0.698132 0.0 0.0 -> xyz=-0.0114 -0.1 0.407 rpy=-0.698132 0.0 0.0

File: alex_description/urdf/20240819_Alex_FixedSpine_FlatHands.urdf (robot description, URDF)
Before this commit: robot Alex, 27 links, 26 joints
Joints:
- joint LeftShoulderPitch: origin xyz=-0.0114 0.1 0.570 rpy=0.698132 0.0 0.0 -> xyz=-0.0114 0.1 0.407 rpy=0.698132 0.0 0.0
- joint NeckYaw: origin xyz=0.000094 -0.000003 0.625793 rpy=0 0 0 -> xyz=0.000094 -0.000003 0.462793 rpy=0 0 0
- joint RightShoulderPitch: origin xyz=-0.0114 -0.1 0.570 rpy=-0.698132 0.0 0.0 -> xyz=-0.0114 -0.1 0.407 rpy=-0.698132 0.0 0.0
