Commit message: Updated Spine based URDF

File: alex_description/urdf/20240808_Alex_Nubs.urdf (robot description, URDF)
Before this commit: robot Alex, 30 links, 29 joints
Links:
- link Head: mass 1.615 -> 1.677; geometry visual mesh filename=package://alex_description/meshes/ALX02_01_A02_HeadLink.obj
- link NeckYawLink: mass 0.708 -> 1.141; geometry visual mesh filename=package://alex_description/meshes/ALX02_01_A03_NeckLink.obj
- link Pelvis: mass 10.0 -> 4.074; geometry visual mesh filename=package://alex_description/meshes/ALX02_02_A01_BaseLink.obj
- link SpineRollLink: mass 0.44 -> 0.235; geometry visual mesh filename=package://alex_description/meshes/ALX02_02_A05_UJointLink.o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
- link SpineYawLink: mass 0.91 -> 1.839; geometry visual mesh filename=package://alex_description/meshes/ALX02_02_A04_BaseDiffLink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
- link Torso: mass 13.5 -> 17.574; geometry visual mesh filename=package://alex_description/meshes/ALX02_02_A06_TorsoLink.obj
Joints:
- joint LeftShoulderPitch: origin xyz=-0.025 0.1 0.214 rpy=0.698132 0.0 0.0 -> xyz=0 0.12799 0.235694 rpy=0.698132 0.0 0.0
- joint NeckPitch: origin xyz=0.025 -0.027544 0.245212 rpy=0 0 0 -> xyz=0.025 0.01 0.207252 rpy=0 0 0
- joint NeckYaw: origin xyz=0.0 -0.00003 0.275793 rpy=0 0 0 -> xyz=0 0 0.307953 rpy=0 0 0
- joint RightShoulderPitch: origin xyz=-0.025 -0.1 0.214 rpy=-0.698132 0.0 0.0 -> xyz=0 -0.12799 0.235694 rpy=-0.698132 0.0 0.0
- joint SpinePitch: origin xyz=0.12 0.0 0.0 rpy=0 0 0 -> xyz=0 0 0.035 rpy=0 0 0
- joint SpineRoll: origin xyz=-0.08 0 0.12 rpy=0 0 0 -> xyz=-0.015 0 0.0528 rpy=0 0 0
- joint SpineYaw: origin xyz=-0.129 0 0.35 rpy=0 0 0 -> xyz=0 0 0.1045 rpy=0 0 0

Commit message: Updated left and right J1 IMU locations and added the Neck yaw IMU to the torso

File: alex_description/urdf/20240808_Alex_Nubs.urdf (robot description, URDF)
Before this commit: robot Alex, 30 links, 29 joints
Links:
- added link NeckBaseIMULink, mass 0
Joints:
- added joint NeckBaseIMUJoint: type fixed, parent Torso, child NeckBaseIMULink, origin xyz=0.00399725 -0.01225021 0.24512039 rpy=0 0 -1.5707963267948966, axis 0 0 1
- joint SpinePitch: limit lower=-0.523599 upper=1.0472 effort=250.0 velocity=6.0 -> lower=-0.523599 upper=0.785398 effort=250.0 velocity=6.0
- joint TorsoLeftIMUJoint: origin xyz=-0.102655 0.034047 0.488646 rpy=1.570796 0 -1.570796 -> xyz=0.07978495 0.10932294  0.17623744 rpy=1.5707963267948966 -0.6981317007977316 1.5707963267948961; parent Pelvis -> Torso
- joint TorsoRightIMUJoint: origin xyz=-0.105655 -0.059053 0.488646 rpy=1.570796 0 -1.570796 -> xyz=0.07978495 -0.09055680 0.16048643 rpy=1.5707963267948966 0.6981317007977319 1.5707963267948966; parent Pelvis -> Torso

Commit message: Debugging on spine testbed for velocity mismatch
The jacobian based velocities do not match with the IMU based velocities

File: alex_description/urdf/20240808_Alex_Nubs.urdf (robot description, URDF)
Before this commit: robot Alex, 30 links, 29 joints
Joints:
- joint SpinePitch: limit lower=-0.523599 upper=1.0472 effort=250.0 velocity=6.0 -> lower=-0.523599 upper=0.785398 effort=250.0 velocity=6.0

Commit message: Updating Alex with nubs robot model to be without the head

File: alex_description/urdf/20240808_Alex_Nubs.urdf (robot description, URDF)
Before this commit: robot Alex, 30 links, 29 joints
Links:
- removed link Head
- removed link NeckYawLink
- removed link TorsoLeftIMULink
- removed link TorsoRightIMULink
- added link TorsoIMULink, mass 0
Joints:
- removed joint NeckPitch
- removed joint NeckYaw
- removed joint TorsoLeftIMUJoint
- removed joint TorsoRightIMUJoint
- added joint TorsoIMUJoint: type fixed, parent Torso, child TorsoIMULink, origin xyz=-0.105655 -0.059053 0.488646 rpy=1.570796 0 -1.570796, axis 0 0 1

Commit message: Adjusted nubs urdf. Will replace with Khizar's version when finished.

File: alex_description/urdf/20240808_Alex_Nubs.urdf (robot description, URDF)
Before this commit: robot Alex, 31 links, 30 joints
Joints:
- joint SpineYaw: type revolute -> fixed

Commit message: Updated URDFs and joint maps

File: alex_description/urdf/20240808_Alex_Nubs.urdf (robot description, URDF)
Before this commit: robot Alex, 27 links, 26 joints
Links:
- removed link TorsoIMULink
- added link Head, mass 1.677; visual mesh filename=package://alex_description/meshes/ALX02_01_A02_HeadLink.obj
- added link NeckBaseIMULink, mass 0
- added link NeckYawLink, mass 1.141; visual mesh filename=package://alex_description/meshes/ALX02_01_A03_NeckLink.obj
- added link TorsoLeftIMULink, mass 0
- added link TorsoRightIMULink, mass 0
Joints:
- removed joint TorsoIMUJoint
- added joint NeckBaseIMUJoint: type fixed, parent Torso, child NeckBaseIMULink, origin xyz=0.00399725 -0.01225021 0.24512039 rpy=0 0 -1.5707963267948966, axis 0 0 1
- added joint NeckPitch: type revolute, parent NeckYawLink, child Head, origin xyz=0.025 0.01 0.207252 rpy=0 0 0, axis 0 1 0, limit lower=-1.0472 upper=1.0472 effort=20 velocity=20
- added joint NeckYaw: type revolute, parent Torso, child NeckYawLink, origin xyz=0 0 0.307953 rpy=0 0 0, axis 0 0 1, limit lower=-1.5708 upper=1.5708 effort=20 velocity=20
- added joint TorsoLeftIMUJoint: type fixed, parent Torso, child TorsoLeftIMULink, origin xyz=0.07978495 0.10932294 0.17623744 rpy=1.5707963267948966 -0.6981317007977316 1.5707963267948961, axis 0 0 1
- added joint TorsoRightIMUJoint: type fixed, parent Torso, child TorsoRightIMULink, origin xyz=0.07978495 -0.09055680 0.16048643 rpy=1.5707963267948966 0.6981317007977319 1.5707963267948966, axis 0 0 1

File: alex_description/urdf/20240929_Alex_SpineTestBed_WithoutHead_SakeHands.urdf (robot description, URDF)
Before this commit: robot Alex, 36 links, 35 joints
Links:
- removed link TorsoIMULink
- added link TorsoLeftIMULink, mass 0
- added link TorsoRightIMULink, mass 0
Joints:
- removed joint TorsoIMUJoint
- added joint TorsoLeftIMUJoint: type fixed, parent Torso, child TorsoLeftIMULink, origin xyz=0.07978495 0.10932294 0.17623744 rpy=1.5707963267948966 -0.6981317007977316 1.5707963267948961, axis 0 0 1
- added joint TorsoRightIMUJoint: type fixed, parent Torso, child TorsoRightIMULink, origin xyz=0.07978495 -0.09055680 0.16048643 rpy=1.5707963267948966 0.6981317007977319 1.5707963267948966, axis 0 0 1
- joint SpineYaw: type revolute -> fixed
