Commit message: Adjusted the urdf.

File: alex_description/urdf/20241003_Alex_SoftwareLockedSpine_LeftSake_RightBarrettWithWeight.urdf (robot description, URDF)
Before this commit: robot Alex, 39 links, 38 joints
Links:
- removed link RightSakeBaseFingerLink1
- removed link RightSakeBaseFingerLink2
- removed link RightSakeFingerTip1
- removed link RightSakeFingerTip2
- removed link RightSakePalmLink
- added link RightBarrettPalmLink, mass 0.944; visual mesh filename=package://barrett_description/meshes/bh280/hand_base.dae
- added link RightHandDumbbellLink, mass 3.956
- added link bh280/finger0_0, mass 0.14109; collision mesh filename=package://barrett_description/meshes/bh280/finger0_0_collis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; visual mesh filename=package://barrett_description/meshes/bh280/finger0_0.dae
- added link bh280/finger0_1, mass 0.062139; collision mesh filename=package://barrett_description/meshes/bh280/finger0_1_collis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; visual mesh filename=package://barrett_description/meshes/bh280/finger0_1.dae
- added link bh280/finger0_2, mass 0.04166; collision mesh filename=package://barrett_description/meshes/bh280/finger0_2_collis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; visual mesh filename=package://barrett_description/meshes/bh280/finger0_2.dae
- added link bh280/finger1_0, mass 0.14109; collision mesh filename=package://barrett_description/meshes/bh280/finger1_0_collis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; visual mesh filename=package://barrett_description/meshes/bh280/finger1_0.dae
- added link bh280/finger1_1, mass 0.062139; collision mesh filename=package://barrett_description/meshes/bh280/finger1_1_collis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; visual mesh filename=package://barrett_description/meshes/bh280/finger1_1.dae
- added link bh280/finger1_2, mass 0.04166; collision mesh filename=package://barrett_description/meshes/bh280/finger1_2_collis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; visual mesh filename=package://barrett_description/meshes/bh280/finger1_2.dae
- added link bh280/finger2_1, mass 0.062139; collision mesh filename=package://barrett_description/meshes/bh280/finger2_1_collis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; visual mesh filename=package://barrett_description/meshes/bh280/finger2_1.dae
- added link bh280/finger2_2, mass 0.04166; collision mesh filename=package://barrett_description/meshes/bh280/finger2_2_collis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; visual mesh filename=package://barrett_description/meshes/bh280/finger2_2.dae
- added link bh280/hand_base, mass 0.60858; collision mesh filename=package://barrett_description/meshes/bh280/hand_base_collis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; visual mesh filename=package://barrett_description/meshes/bh280/hand_base.dae
Joints:
- removed joint RightSakeKnuckle1
- removed joint RightSakeKnuckle2
- removed joint Right_GRIPPER_X1
- removed joint Right_GRIPPER_X2
- added joint RightHandDumbbellAttachmentFixedJoint: type fixed, parent RightBarrettPalmLink, child RightHandDumbbellLink, origin xyz=0 0 -0.027 rpy=0 0 0
- added joint bh280/j00: type fixed, parent bh280/hand_base, child bh280/finger0_0, origin xyz=-0.025 0 0.0754000000000003 rpy=-9.27906974436996E-30 -2.56739074444568E-16 -1.5707963267949, axis 0 0 -1, limit lower=0 upper=3.14159265359 effort=0 velocity=2.0
- added joint bh280/j01: type fixed, parent bh280/finger0_0, child bh280/finger0_1, origin xyz=0.0500000000000007 0.000799999999999971 0 rpy=1.5707963267949 0 0, axis 0 0 1, limit lower=0 upper=2.44346095279 effort=0 velocity=2.0
- added joint bh280/j02: type fixed, parent bh280/finger0_1, child bh280/finger0_2, origin xyz=0.069935684739622 0.00300000000000003 0.000200000000006934 rpy=-3.77533479986348E-14 -4.45260733378639E-14 0.698131700822416, axis 0 0 1, limit lower=0 upper=0.837758040957 effort=0 velocity=2.0, mimic joint=bh280/j01 multiplier=0.321428571429 offset=0.0
- added joint bh280/j10: type fixed, parent bh280/hand_base, child bh280/finger1_0, origin xyz=0.025 0 0.0754 rpy=-9.2871E-30 -0.0058448 -1.5708, axis 0.0058448 0 0.99998, limit lower=0 upper=3.14159265359 effort=0 velocity=2.0, mimic joint=bh280/j00 multiplier=1 offset=0
- added joint bh280/j11: type fixed, parent bh280/finger1_0, child bh280/finger1_1, origin xyz=0.0499991459461259 0.000799999999999367 -0.000292240753933679 rpy=1.5707963267949 0 -4.93038065763132E-32, axis 0 0 1, limit lower=0 upper=2.44346095279 effort=0 velocity=2.0
- added joint bh280/j12: type fixed, parent bh280/finger1_1, child bh280/finger1_2, origin xyz=0.0699356847396015 0.00300000000003377 0.000199999999999378 rpy=1.95799899548702E-16 2.29686057908074E-16 0.700079983587682, axis 0 0 1, limit lower=0 upper=0.837758040957 effort=0 velocity=2.0, mimic joint=bh280/j11 multiplier=0.321428571429 offset=0.0
- added joint bh280/j21: type fixed, parent bh280/hand_base, child bh280/finger2_1, origin xyz=-0.000799999999999992 0.05 0.0754000000000003 rpy=1.5707963267949 2.77555756156289E-17 1.5707963267949, axis 0 0 1, limit lower=0 upper=2.44346095279 effort=0 velocity=2.0
- added joint bh280/j22: type fixed, parent bh280/finger2_1, child bh280/finger2_2, origin xyz=0.0699356847396236 0.00300000000000011 0.000199999999999993 rpy=5.6276902721421E-16 5.75421399737176E-16 0.698131700797743, axis 0 0 1, limit lower=0 upper=0.837758040957 effort=0 velocity=2.0, mimic joint=bh280/j21 multiplier=0.321428571429 offset=0.0
- joint RightGrippertAttachmentFixedJoint: child RightSakePalmLink -> RightBarrettPalmLink
