Commit message: Refactored the fixed spine URDF to include the head

File: alex_description/urdf/20241001_Alex_SoftwareLockedSpine_SakeHands.urdf (robot description, URDF)
Before this commit: robot Alex, 37 links, 36 joints
Links:
- added link Head, mass 1.677; visual mesh filename=package://alex_description/meshes/ALX02_01_A02_HeadLink.obj
- added link NeckYawLink, mass 1.141; visual mesh filename=package://alex_description/meshes/ALX02_01_A03_NeckLink.obj
Joints:
- added joint NeckPitch: type revolute, parent NeckYawLink, child Head, origin xyz=0.025 0.01 0.207252 rpy=0 0 0, axis 0 1 0, limit lower=-1.0472 upper=1.0472 effort=20 velocity=20
- added joint NeckYaw: type revolute, parent Torso, child NeckYawLink, origin xyz=0 0 0.307953 rpy=0 0 0, axis 0 0 1, limit lower=-1.5708 upper=1.5708 effort=20 velocity=20

Commit message: Changed NeckBase IMU name to TorsoIMU

File: alex_description/urdf/20241001_Alex_SoftwareLockedSpine_SakeHands.urdf (robot description, URDF)
Before this commit: robot Alex, 39 links, 38 joints
Links:
- removed link NeckBaseIMULink
- added link TorsoIMULink, mass 0
Joints:
- removed joint NeckBaseIMUJoint
- added joint TorsoIMUJoint: type fixed, parent Torso, child TorsoIMULink, origin xyz=0.00399725 -0.01225021 0.24512039 rpy=0 0 -1.5707963267948966, axis 0 0 1
