Commit message: Moved most of the urdfs to backup. Will make a branch to save them and then delete most of them.

File: alex_description/urdf_backup/20240808_Alex_Nubs_OLD.urdf (robot description, URDF)
Before this commit: robot Alex, 39 links, 38 joints
Links:
- removed link LeftSakeBaseFingerLink1
- removed link LeftSakeBaseFingerLink2
- removed link LeftSakeFingerTip1
- removed link LeftSakeFingerTip2
- removed link LeftSakePalmLink
- removed link RightSakeBaseFingerLink1
- removed link RightSakeBaseFingerLink2
- removed link RightSakeFingerTip1
- removed link RightSakeFingerTip2
- removed link RightSakePalmLink
- removed link TorsoIMULink
- added link NeckBaseIMULink, mass 0
- added link leftNub, mass 0.1; visual mesh filename=package://alex_description/meshes/cycloidal_arm/nub.obj
- added link rightNub, mass 0.1; visual mesh filename=package://alex_description/meshes/cycloidal_arm/nub.obj
Joints:
- removed joint LeftSakeKnuckle1
- removed joint LeftSakeKnuckle2
- removed joint Left_GRIPPER_X1
- removed joint Left_GRIPPER_X2
- removed joint RightSakeKnuckle1
- removed joint RightSakeKnuckle2
- removed joint Right_GRIPPER_X1
- removed joint Right_GRIPPER_X2
- removed joint TorsoIMUJoint
- added joint NeckBaseIMUJoint: type fixed, parent Torso, child NeckBaseIMULink, origin xyz=0.00399725 -0.01225021 0.24512039 rpy=0 0 -1.5707963267948966, axis 0 0 1
- joint LeftGrippertAttachmentFixedJoint: child LeftSakePalmLink -> leftNub
- joint RightGrippertAttachmentFixedJoint: child RightSakePalmLink -> rightNub
